File: ch32-breakout.kicad_sch (KiCad schematic)
At the start: 37 parts, among them J1 Conn_ARM_SWD_TagConnect_TC203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, J2 USB_C_Receptacle_USB2.0_16P, J3 Conn_01x05_Socket, J4 Conn_01x05_Socket, J5 Conn_01x05_Socket, J6 Conn_01x05_Socket, Q1 Q_Dual_PMOS_S1G1D2S2G2D1, U1 CH32V003FxUx, U2 TP4057, U3 XB3303ASOT23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

Commit message: Bpard finished it's kibot time
Parts:
- D1: LCSC Part (none) -> C5336761
- J2: LCSC Part (none) -> C319148
- R1: LCSC Part (none) -> C60490
- R10: LCSC Part (none) -> C106232
- R2, R7: LCSC Part (none) -> C2929900
- R3, R4: LCSC Part (none) -> C103086
- R5, R6: LCSC Part (none) -> C137973
- R8, R9: LCSC Part (none) -> C2906883
Changed lines of the file:
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@@
 			)
 		)
-		(property "LCSC Part" ""
+		(property "LCSC Part" "C106232 "
 			(at 140.97 101.6 0)
 			(effects
@@
 			)
 		)
-		(property "LCSC Part" ""
+		(property "LCSC Part" "C2906883"
 			(at 116.84 63.5 0)
 			(effects
@@
 			)
 		)
-		(property "LCSC Part" ""
+		(property "LCSC Part" "C2906883"
 			(at 118.11 80.01 0)
 			(effects
@@
 			)
 		)
-		(property "LCSC Part" ""
+		(property "LCSC Part" "C2929900"
 			(at 90.17 148.59 0)
 			(effects
@@
 			)
 		)
-		(property "LCSC Part" ""
+		(property "LCSC Part" "C137973"
 			(at 90.17 156.21 0)
 			(effects
@@
 			)
 		)
-		(property "LCSC Part" ""
+		(property "LCSC Part" "C319148"
 			(at 66.04 152.4 0)
 			(effects
@@
 			)
 		)
-		(property "LCSC Part" ""
+		(property "LCSC Part" "C5336761"
 			(at 63.5 106.68 0)
 			(effects
@@
 			)
 		)
-		(property "LCSC Part" ""
+		(property "LCSC Part" "C137973"
 			(at 90.17 151.13 0)
 			(effects
@@
 			)
 		)
-		(property "LCSC Part" ""
+		(property "LCSC Part" "C103086"
 			(at 90.17 144.78 0)
 			(effects
@@
 			)
 		)
-		(property "LCSC Part" ""
+		(property "LCSC Part" "C2929900"
 			(at 58.42 110.49 0)
 			(effects
@@
 			)
 		)
-		(property "LCSC Part" ""
+		(property "LCSC Part" "C60490"
 			(at 78.74 123.19 0)
 			(effects
@@
 			)
 		)
-		(property "LCSC Part" ""
+		(property "LCSC Part" "C103086"
 			(at 90.17 142.24 0)
 			(effects
